File: pcb/mk2/mk2.kicad_sch (KiCad schematic)
At the start: 0 parts

Commit message: Updated symbol library for PCB.
Parts:
- added U1: (no value), symbol mk2:TEENSY41
Changed lines of the file:
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@@
 	(generator_version "10.0")
 	(paper "A4")
+	(symbol
+		(lib_id "mk2:TEENSY41")
+		(at 101.6 101.6 0)
+		(unit 1)
+		(body_style 1)
+		(exclude_from_sim no)
+		(in_bom yes)
+		(on_board yes)
+		(in_pos_files yes)
+		(dnp no)
+		(fields_autoplaced yes)
+		(property "Reference" "U1"
+			(at 103.7433 90.17 0)
+			(show_name no)
+			(do_not_autoplace no)
+			(effects
+				(font
+					(size 1.27 1.27)
+				)
+				(justify left)
+			)
+		)
+		(property "Value" ""
+			(at 101.6 101.6 0)
+			(show_name no)
+			(do_not_autoplace no)
+			(effects
+				(font
+					(size 1.27 1.27)
+				)
+			)
+		)
+		(property "Footprint" ""
+			(at 101.6 101.6 0)
+			(hide yes)
+			(show_name no)
+			(do_not_autoplace no)
+			(effects
+				(font
+					(size 1.27 1.27)
+				)
+			)
+		)
+		(property "Datasheet" ""
+			(at 101.6 101.6 0)
+			(hide yes)
+			(show_name no)
+			(do_not_autoplace no)
+			(effects
+				(font
+					(size 1.27 1.27)
+				)
+			)
+		)
+		(property "Description" ""
+			(at 101.6 101.6 0)
+			(hide yes)
+			(show_name no)
+			(do_not_autoplace no)
+			(effects
+				(font
+					(size 1.27 1.27)
+				)
+			)
+		)
+		(pin "Vin"
+		)
+		(pin "4"
+		)
+		(pin "36"
+		)
+		(pin "39"
+		)
+		(pin "3"
+		)
+		(pin "41"
+		)
+		(pin "2"
+		)
+		(pin "5"
+		)
+		(pin "40"
+		)
+		(pin "3.3V"
+		)
+		(pin "GND"
+		)
+		(pin "37"
+		)
+		(pin "38"
+		)
+		(instances
+			(project "mk2"
+				(path "/6101f0c6-c055-4fd8-8ef5-35c06105f18c"
+					(reference "U1")
+					(unit 1)
+				)
+			)
+		)
+	)
 	(sheet_instances
 		(path "/"
